File: kicad/tars4.kicad_sch (KiCad schematic)
At the start: 56 parts, among them J2 microSD (jambe G), Q1 AO3401A, Q5 AO3401A, SW1 inter. ≥ 1 A, U1 TP4056 + DW01, R_PROG 2,4k, U10 AM312, U11 BME280 (jambe D), U2 LOLIN S3 Mini, U3 Écran 1 (milieu G), U4 Écran 2 (milieu D), U5 MAX98357A (milieu D), U6 INMP441 (milieu G), U7 DS3231 ZS-042 (jambe D), U8 ADXL345 GY-291, U9 TPS63020 3,3 V

Commit message: docs: translate the KiCad schematic notes and labels to English (kicad_sch_gen.py, schematic, PDF)
Co-Authored-By: Claude Opus 5.5 <noreply@anthropic.com>
Parts:
- J2: value microSD (jambe G) -> microSD (left leg)
- R12, R19: value 47 (support) -> 47 (carrier)
- R20: value 33 (support) -> 33 (carrier)
- U11: value BME280 (jambe D) -> BME280 (right leg)
- U3: value Écran 1 (milieu G) -> Screen 1 (left middle)
- U4: value Écran 2 (milieu D) -> Screen 2 (right middle)
- U5: value MAX98357A (milieu D) -> MAX98357A (right middle)
- U6: value INMP441 (milieu G) -> INMP441 (left middle)
- U7: value DS3231 ZS-042 (jambe D) -> DS3231 ZS-042 (right leg)
Other:
- note added: "BL_EN (GPIO7): backlight of both screens only (PWM possible). AMP_SD (GPIO4): R10 1k + R18 10k on P2 → amplifier SD (off at boot and in sleep). P1 / P2: stripboards under the screens. I2C chain: S3 → ADXL345 → middle tube → P2 → right tube → DS3231 + BME280 (right leg); sensor supply P1 → mic → ADXL345, P2 → right leg."
- note added: "BRAIN — LOLIN S3 Mini (left middle)"
- note added: "C1 (SMD 7343 tantalum lying under the S3) on its carrier, C2 / C3 on the P1 3V3 strip, C10 / C11 on P2; plans renders/tars4_board_*.svg."
- note added: "Connectors X1–X15 (keyed Dupont / JST) between each module and the harness, S3 plugged into a carrier: not drawn, see tars4_wiring.html. D3: unidirectional TVS (Zener symbol). A crossing without a dot is not a connection. Generated by tools/kicad_sch_gen.py (netlist checked at every generation)."
- note added: "LEDs: remove every status LED fed by the battery (ZS-042, TPS63020, GY-291, microSD reader…); keep the TP4056 charge LEDs."
- note added: "POWER — ground star on the power-path board (left leg)"
- note added: "Q1 + D1 + R1: power path (mains / battery). R2 / R3 (1M, on B+: the real cell voltage, even on mains) on the power-path board; C6 (GPIO1) and C8 (GPIO21) at the S3 pins. Q5 + R22 on the power-path board: microSD cut in sleep (GPIO36 low = on)."
- note added: "R15 / R16: charger plugged in → USB_DET ≈ 3 V (GPIO21, wake-up)."
- note added: "S3: V (VBUS) = the S3 USB-C only. EN = S3 reset (≠ BL_EN). 33 Ω series at the S3 (R20 on MOSI); SCK split on the carrier: R12 → screen 1, R19 → screen 2 (direct wire in the tube), 47 Ω (up to 100 if the image jitters)."
- note added: "SCREENS, I2C SENSORS →"
- note added: "SOUND, MIC, microSD"
- note added: "Silicone wire: power in 26 AWG (B+/B−, amplifier pair, 3V3 and GND to P1), signals and screen / sensor supply in 30 AWG. Tubes: 13 / 19 / 6 wires."
- note added: "U10: front hole at the top (right middle), R17 on P2; U7, U11 in the right leg (SQW not wired)."
- note added: "U9: EN tied to VIN, PS/SYNC to GND (never drive it high). Its VSYS/GND pair leaves from the star; the logic GND to P1 leaves from its GND pad."
- note added: "VUSB (J1: micro-USB breakout at the foot of the left leg; D3 + C9 on the TP4056 IN pads)"
- note removed: "ALIMENTATION — étoile de masse sur la plaquette du partage de charge (jambe G)"
- note removed: "BL_EN (GPIO7) : rétroéclairage des deux écrans seulement (PWM possible). AMP_SD (GPIO4) : R10 1k + R18 10k sur P2 → SD de l'ampli (éteint au démarrage et en veille). P1 / P2 : plaques à bandes sous les écrans. I2C en chaîne : S3 → ADXL345 → tube central → P2 → tube droit → DS3231 + BME280 (jambe D) ; alim des capteurs P1 → micro → ADXL345, P2 → jambe D."
- note removed: "C1 (tantale CMS 7343 couché sous la S3) sur son support, C2 / C3 sur la bande 3V3 de P1, C10 / C11 sur P2 ; plans renders/tars4_board_*.svg."
- note removed: "CERVEAU — LOLIN S3 Mini (milieu G)"
- note removed: "Connecteurs X1–X15 (Dupont détrompés / JST) entre chaque module et le faisceau, S3 enfichée sur un support : non dessinés, voir tars4_wiring.html. D3 : TVS unidirectionnelle (symbole Zener). Un croisement sans point n'est pas une connexion. Généré par tools/kicad_sch_gen.py (netlist vérifiée à chaque génération)."
- note removed: "Fils silicone : alimentation en 26 AWG (B+/B−, paire ampli, 3V3 et GND vers P1), signaux et alimentation des écrans / capteurs en 30 AWG. Tubes : 13 / 19 / 6 fils."
- note removed: "LED : retirer toutes les LED d'état alimentées par la batterie (ZS-042, TPS63020, GY-291, lecteur microSD…) ; garder celles de charge du TP4056."
- note removed: "Q1 + D1 + R1 : partage de charge (secteur / batterie). R2 / R3 (1M, sur B+ : la vraie tension des cellules, même sur secteur) sur la plaquette ; C6 (GPIO1) et C8 (GPIO21) aux broches de la S3. Q5 + R22 sur la plaquette : microSD coupée en veille (GPIO36 bas = allumée)."
- note removed: "R15 / R16 : chargeur branché → USB_DET ≈ 3 V (GPIO21, réveil)."
- note removed: "S3 : V (VBUS) = USB-C de la S3 seulement. EN = reset de la S3 (≠ BL_EN). Séries 33 Ω côté S3 (R20 sur MOSI) ; SCK séparé sur le support : R12 → écran 1, R19 → écran 2 (fil direct dans le tube), 47 Ω (jusqu'à 100 si l'image sautille)."
- note removed: "SON, MICRO, microSD"
- note removed: "U10 : trou en façade en haut (milieu D), R17 sur P2 ; U7, U11 dans la jambe D (SQW non câblé)."
- note removed: "U9 : EN relié à VIN, PS/SYNC à GND (ne jamais le mettre à l'état haut). Sa paire VSYS/GND part de l'étoile ; le GND logique vers P1 part de sa pastille GND."
- note removed: "VUSB (J1 : breakout micro-USB au pied de la jambe G ; D3 + C9 sur les pastilles IN du TP4056)"
- note removed: "ÉCRANS, CAPTEURS I2C →"
- title: TARS4 — électronique -> TARS4 — electronics
