File: hardware/kicad/tars4.kicad_sch (KiCad schematic)
At the start: 56 parts, among them J2 microSD (left leg), Q1 AO3401A, Q5 AO3401A, SW1 inter. ≥ 1 A, U1 TP4056 + DW01, R_PROG 2,4k, U10 AM312, U11 BME280 (right leg), U2 LOLIN S3 Mini, U3 Screen 1 (left middle), U4 Screen 2 (right middle), U5 MAX98357A (right middle), U6 INMP441 (left middle), U7 DS3231 ZS-042 (right leg), U8 ADXL345 GY-291, U9 TPS63020 3,3 V

Commit message: fix(PLAT-POWER-CHARGE-001): J1, the micro-USB charging socket, drawn in the schematic
J1 was only a text note, so the netlist had no breakout and the requirement's acceptance (its VBUS / GND on the TP4056
IN+ / IN- pads) could not be checked. New module symbol tars:usb_charging_socket (VBUS, GND; usbb in tars4.scad) on
VUSB and GND; the note now says "heel" (the port moved there in mech-usb-heel). Netlist check OK (49 nets), ERC
clean, schematic PDF exported; the acceptance test loses its xfail mark.

Co-Authored-By: Claude Opus 5.5 <noreply@anthropic.com>
Parts:
- removed C6: 0.1µ (S3), symbol Device:C
- removed C7: 470µ 10V, symbol Device:C_Polarized
- removed Q1: AO3401A, symbol Device:Q_PMOS
- removed U8: ADXL345 GY-291, symbol tars:ADXL345_GY-291
- removed U9: TPS63020 3,3 V, symbol tars:TPS63020_3V3
- added BT2: 18650 D, symbol Device:Battery_Cell
- added C8: 0.1µ (S3), symbol Device:C
- added R16: 100k, symbol Device:R
- added R5: 10k, symbol Device:R
- added SW1: inter. ≥ 1 A, symbol Switch:SW_SPST
- added U11: BME280 (right leg), symbol tars:BME280_GY
- BT1: renamed from BT2; value 18650 D -> 18650 G
- C7: renamed from R5; value 10k -> 470µ 10V; symbol Device:R -> Device:C_Polarized
- D1: renamed from SW1; value inter. ≥ 1 A -> 1N5822; symbol Switch:SW_SPST -> Device:D_Schottky
- F2: renamed from BT1; value 18650 G -> PPTC 1.6A; symbol Device:Battery_Cell -> Device:Polyfuse
- J1: renamed from R15; value 68k -> USB charging socket; symbol Device:R -> tars:usb_charging_socket
- Q1: renamed from D1; value 1N5822 -> AO3401A; symbol Device:D_Schottky -> Device:Q_PMOS
- R15: renamed from R16; value 100k -> 68k
- R3: renamed from F1; value PPTC 1.6A -> 1M; symbol Device:Polyfuse -> Device:R
- U8: renamed from U11; value BME280 (right leg) -> ADXL345 GY-291; symbol tars:BME280_GY -> tars:ADXL345_GY-291
- U9: renamed from R2; value 1M -> TPS63020 3,3 V; symbol Device:R -> tars:TPS63020_3V3
- renumbered C8 to C6, F2 to F1, R3 to R2
Connections:
- net +3V3: now also U8.CS, U9.VOUT, U11.VCC
- net GND: now also C7.2, J1.GND, R3.2, U8.SDO, U9.GND, U9.PS, C8.2, R16.2, U11.GND; no longer R15.2, R2.2
- net SD_3V3: now also R5.1; no longer C7.1
- net USB_DET: now also R15.2, C8.1, R16.1; no longer C6.1, J1.2, R15.1
- net at U2.6 (IO6), U7.SCL, U8.SCL: now also U11.SCL
- net at U2.5 (IO5), U7.SDA, U8.SDA: now also U11.SDA
- net at U5.VIN: now also C7.1, U9.EN, U9.VIN, SW1.2 (B); no longer D1.2 (B)
- net at J2.CMD, U2.34 (IO34): now also R5.2; no longer C7.2
- net at D1.1 (K): now also Q1.S, SW1.1 (A); no longer Q1.1 (K)
- net at U2.2 (IO2): now also U8.INT1
- net at C9.1, D3.1 (K), R1.1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: now also D1.2 (A), J1.VBUS, Q1.G, R15.1; no longer J1.1, Q1.2 (A)
- net at BT1.2 (-), U1.B-: now also BT2.2 (-); no longer F2.2 (-)
- net at F2.1: now also F1.1, R2.1, U1.B+; no longer R3.2
- net at U1.OUT+: now also Q1.D
- new net: BT2.1 (+), F2.2
- new net: C6.1, R2.2, R3.1, U2.1 (IO1)
Other:
- note added: "VUSB (J1: micro-USB charging socket at the heel of the left leg; D3 + C9 on the TP4056 IN pads)"
- note removed: "VUSB (J1: micro-USB breakout at the foot of the left leg; D3 + C9 on the TP4056 IN pads)"
- moved on the sheet: BT1, C6, F1, R15, R2

Commit message: feat(PLAT-POWER-VSENSE-001): Q4 BC547B, R23 / R24 1 MΩ and GPIO37 in the schematic
VSYS → R23 → base, R24 base → GND, emitter GND, collector on GPIO37 (VSENSE), drawn as a block joined by labels. Netlist OK (51 nets), ERC clean; the acceptance test loses its xfail mark.

Co-Authored-By: Claude Opus 5.5 <noreply@anthropic.com>
Parts:
- removed R6, R8, R9: 10k, symbol Device:R
- added C4: 10µ tant., symbol Device:C_Polarized
- added C5: 0.1µ, symbol Device:C
- added R22: 100k, symbol Device:R
- added R23: 1M (harness, P4 end), symbol Device:R
- added R24: 1M (carrier), symbol Device:R
- added R5: 10k, symbol Device:R
- Q4: renamed from R5; value 10k -> BC547B (carrier); symbol Device:R -> Device:Q_NPN
- R6: renamed from R22; value 100k -> 10k
- R8: renamed from C4; value 10µ tant. -> 10k; symbol Device:C_Polarized -> Device:R
- R9: renamed from C5; value 0.1µ -> 10k; symbol Device:C -> Device:R
Connections:
- net +3V3: now also R22.1; no longer R6.1
- net GND: now also Q4.E, C4.2, C5.2, R24.2; no longer R8.2, R9.2
- net SD_3V3: now also R6.1, C4.1, C5.1, R5.1; no longer Q4.1
- net VSYS: now reaches C7.1, SW1.2 (B), U5.VIN, U9.EN, U9.VIN
- net VSYS: now also R23.1
- net at J2.D3: now also R9.2
- net at Q5.G, U2.36 (IO36): now also R22.2; no longer R6.2
- net at J2.D0, U2.35 (IO35): now also R6.2
- net at J2.CMD, U2.34 (IO34): now also R5.2; no longer Q4.2
- net VSENSE: now reaches U2.37 (IO37)
- net VSENSE: now also Q4.C
- net at J2.D2: now also R8.2
- new net: Q4.B, R23.2, R24.1
- no-connect marks 9 -> 8
Other:
- note added: "Silicone wire: power in 26 AWG (B+/B−, amplifier pair, 3V3 and GND to P1), signals and screen / sensor supply in 30 AWG. Tubes: 14 / 19 / 6 wires."
- note added: "VSYS SENSE — R23 in the harness at P4, R24 + Q4 on the carrier: GPIO37 low = VSYS present"
- note removed: "Silicone wire: power in 26 AWG (B+/B−, amplifier pair, 3V3 and GND to P1), signals and screen / sensor supply in 30 AWG. Tubes: 13 / 19 / 6 wires."
- moved on the sheet: R6

Commit message: feat(PLAT-POWER-MONITOR-001): R2 in line in the harness at the TP4056 B+ pad, R3 on the power-path board
The sense wire carried raw B+ in 30 AWG behind the polyfuses only; it now carries B+ behind 1 MΩ. P4 loses R2 and its B+ hole (J5–J8 free); boards.py / harness.py learn in-line resistors at the far end of a wire. Schematic regenerated (netlist OK, 51 nets), PDF, board plans, harness guide and wiring SVG updated.

Co-Authored-By: Claude Opus 5.5 <noreply@anthropic.com>
Parts:
- R1: value 10k -> 4.7k
- R2: value 1M -> 1M (harness, B+ pad)
- R24: value 1M (carrier) -> 330k (carrier)
Changed lines of the file:
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@@
 			)
 		)
-		(property "Value" "1M (carrier)"
+		(property "Value" "330k (carrier)"
 			(at 421.64 80.01 0)
 			(show_name no)
@@
 			)
 		)
-		(property "Value" "1M"
+		(property "Value" "1M (harness, B+ pad)"
 			(at 144.78 63.5 0)
 			(show_name no)
@@
 			)
 		)
-		(property "Value" "10k"
+		(property "Value" "4.7k"
 			(at 33.02 48.26 0)
 			(show_name no)
